Commit message: 例行更新

File: brain/ros2_ws/src/description/urdf/ascamera.xacro (robot description, xacro)
@@ -1,5 +1,6 @@
 <?xml version="1.0" encoding="utf-8"?>
 <robot xmlns:xacro="http://ros.org/wiki/xacro">
-  <link name="camera_link0">
+  <!-- 深度相机主体 -->
+  <link name="depth_camera_link_1">
     <visual>
       <origin xyz="0 0 0" rpy="0 0 0"/>
@@ -8,8 +9,23 @@
     </visual>
   </link>
-  <joint name="depth_camera" type="fixed">
+  <!-- RGB 相机主体 -->
+  <link name="rgb_camera_link_1">
+    <visual>
+      <origin xyz="0 0 0" rpy="0 0 0"/>
+      <geometry><box size="0.02 0.02 0.02"/></geometry>
+      <material name="white"/>
+    </visual>
+  </link>
+  <!-- 深度相机 → base_link -->
+  <joint name="depth_camera_joint_1" type="fixed">
+    <parent link="base_link"/>
+    <child link="depth_camera_link_1"/>
     <origin xyz="0.057373 7.9091E-05 0.091864" rpy="0 0 0"/>
-    <parent link="base_link"/>
-    <child link="camera_link0"/>
+  </joint>
+  <!-- RGB 相机 → depth_camera_link_1 -->
+  <joint name="rgb_camera_joint_1" type="fixed">
+    <parent link="depth_camera_link_1"/>
+    <child link="rgb_camera_link_1"/>
+    <origin xyz="0 0 0" rpy="0 0 0"/>
   </joint>
 </robot>

File: brain/ros2_ws/src/description/urdf/description.urdf.xacro (robot description, xacro)
@@ -1,5 +1,4 @@
 <?xml version="1.0" encoding="utf-8"?>
 <robot name="brain_robot" xmlns:xacro="http://www.ros.org/wiki/xacro">
-  <xacro:property name="camera_type"    value="$(env DEPTH_CAMERA_TYPE)"/>
   <xacro:include filename="$(find description)/urdf/materials.xacro"/>
   <!-- ==================== base_footprint ==================== -->
@@ -152,10 +151,5 @@
     z_offset="0.016719"/>
   <!-- ==================== 深度相机 ==================== -->
-  <xacro:if value="${camera_type == 'AsCamera' or camera_type == 'aurora'}">
-    <xacro:include filename="$(find description)/urdf/ascamera.xacro"/>
-  </xacro:if>
-  <xacro:if value="${camera_type == 'Dabai'}">
-    <xacro:include filename="$(find description)/urdf/dabai.xacro"/>
-  </xacro:if>
+  <xacro:include filename="$(find description)/urdf/ascamera.xacro"/>
   <!-- ==================== ros2_control ==================== -->
   <ros2_control name="BrainSystem" type="system">
